File: 536-counter-7seg/4-digit-clock.sch (EAGLE design)
At the start: 36 parts, among them IC1 SLG46826GTR, IC2 SLG46826GTR, IC3 SLG46826GTR, IC4 SLG46826GTR, IC5 SLG46826GTR, IC7 SLG46826GTR

Commit message: update pcb layouts
Parts:
- SW1: device mylib:TACTSW2-BK-P807X -> mylib:TACTSW2-BK-TL1105S
Connections:
- new net N$51: IC1.IO3, IC7.IO13
- net N$17: now also IC7.IO11; no longer IC7.IO13
- net N$18: now also IC7.IO10; no longer IC7.IO12
- net N$22: now also IC7.IO8; no longer IC7.IO11
- net N$26: now also IC7.IO12
- net N$27: now also IC7.IO9
Other:
- note added: "EXT_RESET(H)"
- note added: "EXT_RESET(M)"
- note added: "EXT_RESET(S)"
- note added: "OPTIONAL"
- moved on the sheet: CON11, CON12, IC1, IC2, IC3, IC4, IC5, LED1, R1, R2, R3, R4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
